File: stm32l031-breakout.sch (KiCad schematic (older format))
At the start: 0 parts

Commit message: MCU symbol
Parts:
- added U?: STM32L031K6Tx, Package_QFP:LQFP-32_7x7mm_P0.8mm, symbol local_symbols:STM32L031K6Tx
Changed lines of the file:
@@
 EESchema Schematic File Version 4
+LIBS:stm32l031-breakout-cache
 EELAYER 26 0
 EELAYER END
@@
 Comment4 ""
 $EndDescr
+$Comp
+L local_symbols:STM32L031K6Tx U?
+U 1 1 5C934203
+P 3400 2700
+F 0 "U?" H 3350 1609 50  0000 C CNN
+F 1 "STM32L031K6Tx" H 3350 1516 50  0000 C CNN
+F 2 "Package_QFP:LQFP-32_7x7mm_P0.8mm" H 2900 1800 50  0001 R CNN
+F 3 "" H 3400 2700 50  0001 C CNN
+	1    3400 2700
+	1    0    0    -1
+$EndComp
 $EndSCHEMATC
