File: stm32l031-breakout.sch (KiCad schematic (older format))
At the start: 1 part

Commit message: Basic schematic
Parts:
- added C? (x4): 0.1uF, symbol Device:C_Small
- added C?: 1uF, symbol Device:C_Small
- added C?: 10uF, symbol Device:C_Small
- added R?: 10k, symbol Device:R
- added SW?: SW_RESET, symbol Switch:SW_Push
- added SW?: SW_BOOT, symbol Switch:SW_Push
Connections:
- net VDD: now reaches U?.1 (VDD)
- net VDD: now also U?.17 (VDD), U?.5 (VDDA), C?.1, C?.1, C?.1, C?.1, C?.1, SW?.2
- net GND: now reaches U?.16 (VSS)
- net GND: now also U?.32 (VSS), C?.2, C?.2, C?.2, C?.2, C?.2, C?.2, R?.2, SW?.1
- net BOOT: now reaches U?.31 (BOOT0)
- net BOOT: now also R?.1, SW?.1
- net at U?.4 (NRST): now also C?.1, SW?.2

Commit message: More schematic, some footprints
Parts:
- added J? (x2): Conn_01x16, symbol Connector_Generic:Conn_01x16
- added J? (x4): Conn_01x01, symbol Connector_Generic:Conn_01x01
- added J?: Conn_01x02, symbol Connector_Generic:Conn_01x02
Connections:
- net GND: now also J?.1 (Pin_1), J?.1 (Pin_1), J?.1 (Pin_1), J?.1 (Pin_1)
- net PA4: now reaches U?.10 (NSS/PA4)
- net PA5.SCK: now reaches U?.11 (SCK/PA5)
- net PA6.MISO: now reaches U?.12 (MISO/PA6)
- net PA7.MOSI: now reaches U?.13 (MOSI/PA7)
- net PB0: now reaches U?.14 (PB0)
- net PB1: now reaches U?.15 (PB1)
- net PA8: now reaches U?.18 (PA8)
- net PA8.SCL.TX: now reaches U?.19 (SCL/TX2/PA9)
- net PC14: now reaches U?.2 (PC14)
- net PA10.SDA.RX: now reaches U?.20 (SDA/RX2/PA10)
- net PA11: now reaches U?.21 (PA11)
- net PA12: now reaches U?.22 (PA12)
- net PA13.SWDIO: now reaches U?.23 (SWDIO/PA13)
- net PA14.SWCLK: now reaches U?.24 (SWCLK/PA14)
- net PA15: now reaches U?.25 (PA15)
- net PB3: now reaches U?.26 (PB3)
- net PB4: now reaches U?.27 (PB4)
- net PB5: now reaches U?.28 (PB5)
- net PB6: now reaches U?.29 (PB6)
- net PC15: now reaches U?.3 (PC15)
- net PB7: now reaches U?.30 (PB7)
- net PA0: now reaches U?.6 (PA0)
- net PA1: now reaches U?.7 (PA1)
- net PA2.TX: now reaches U?.8 (TX2/PA2)
- net PA3.RX: now reaches U?.9 (RX2/PA3)
Other:
- note added: "26 GPIOs\n+1 VDD\n+1 GND\n+4 extra GND\n= 32 pins"
- note added: "BOOT=0: run from flash\nBOOT=1: run bootloader"
- note added: "STM32L031K6T7\n(32-LQFP)\nBreaking out:\n 2 (PC) + 8 (PB) + 16 (PA)\n = 26 pins"
- note added: "additional GND pins"
- note added: "additional caps\nfor VDDA"
- note added: "decoupling cap\nfor each VDD"
- note added: "power supply cap"
- moved on the sheet: C?, R?, SW?

Commit message: Complete schematic
Parts:
- removed J? (x4): Conn_01x01, symbol Connector_Generic:Conn_01x01
- removed J?: Conn_01x02, symbol Connector_Generic:Conn_01x02
- SW_RST: renamed from SW?; value SW_RESET -> SW_RST
- gave numbers to parts that had none: 11
Connections:
- net PA8.SCL.TX is gone; now on net PA9.SCL.TX: U1.19 (SCL/TX2/PA9)
- net GND: now also J1.14 (Pin_14), J1.2 (Pin_2), J1.9 (Pin_9), J2.1 (Pin_1), J2.13 (Pin_13), J2.7 (Pin_7)
- net PA0: now also J1.5 (Pin_5)
- net PA1: now also J1.6 (Pin_6)
- net PA10.SDA.RX: now also J2.14 (Pin_14)
- net PA11: now also J2.12 (Pin_12)
- net PA12: now also J2.11 (Pin_11)
- net PA13.SWDIO: now also J2.10 (Pin_10)
- net PA14.SWCLK: now also J2.9 (Pin_9)
- net PA15: now also J2.8 (Pin_8)
- net PA2.TX: now also J1.7 (Pin_7)
- net PA3.RX: now also J1.8 (Pin_8)
- net PA4: now also J1.10 (Pin_10)
- net PA5.SCK: now also J1.11 (Pin_11)
- net PA6.MISO: now also J1.12 (Pin_12)
- net PA7.MOSI: now also J1.13 (Pin_13)
- net PA8: now also J2.16 (Pin_16)
- net PB0: now also J1.15 (Pin_15)
- net PB1: now also J1.16 (Pin_16)
- net PB3: now also J2.6 (Pin_6)
- net PB4: now also J2.5 (Pin_5)
- net PB5: now also J2.4 (Pin_4)
- net PB6: now also J2.3 (Pin_3)
- net PB7: now also J2.2 (Pin_2)
- net PC14: now also J1.3 (Pin_3)
- net PC15: now also J1.4 (Pin_4)
- net VDD: now also J1.1 (Pin_1)
- net PA9.SCL.TX: now reaches J2.15 (Pin_15)
Other:
- note added: "25 GPIOs\n+1 VDD\n+1 GND\n+5 extra GND\n= 32 pins"
- note added: "STM32L031K6T7\n(32-LQFP)\nBreaking out:\n 2 (PC) + 7 (PB) + 16 (PA)\n = 25 pins"
- note added: "VDD = 1.65V to 3.6V"
- note removed: "26 GPIOs\n+1 VDD\n+1 GND\n+4 extra GND\n= 32 pins"
- note removed: "STM32L031K6T7\n(32-LQFP)\nBreaking out:\n 2 (PC) + 8 (PB) + 16 (PA)\n = 26 pins"
- note removed: "additional GND pins"
- moved on the sheet: C5, J1, J2

Commit message: Footprint tuning, net list, initial PCB placement
Parts:
- C1, C2, C3, C6, R1: footprint (none) -> local_footprints:0805_HS
- C4: footprint (none) -> local_footprints:1206_HS
- C5: footprint (none) -> local_footprints:1210_HS
- J1, J2: footprint (none) -> local_footprints:Pin_Header_Straight_1x16_Pitch2.54mm
- SW_BOOT1: renamed from SW_BOOT; footprint (none) -> local_footprints:SW_SPST_PUSH_6mm_3mm
- SW_RST1: renamed from SW_RST; footprint (none) -> local_footprints:SW_SPST_PUSH_6mm_3mm
- U1: footprint Package_QFP:LQFP-32_7x7mm_P0.8mm -> local_footprints:TQFP-32_7x7mm_Pitch0.8mm_HS_narrow_pads
Changed lines of the file:
@@
 F 0 "U1" H 3550 1650 50  0000 C CNN
 F 1 "STM32L031K6Tx" H 3800 1550 50  0000 C CNN
-F 2 "Package_QFP:LQFP-32_7x7mm_P0.8mm" H 2900 1800 50  0001 R CNN
+F 2 "local_footprints:TQFP-32_7x7mm_Pitch0.8mm_HS_narrow_pads" H 2900 1800 50  0001 R CNN
 F 3 "" H 3400 2700 50  0001 C CNN
 	1    3400 2700
@@
 F 0 "C2" H 2992 1547 50  0000 L CNN
 F 1 "0.1uF" H 2992 1454 50  0000 L CNN
-F 2 "" H 2900 1500 50  0001 C CNN
+F 2 "local_footprints:0805_HS" H 2900 1500 50  0001 C CNN
 F 3 "~" H 2900 1500 50  0001 C CNN
 	1    2900 1500
@@
 F 0 "C1" H 2500 1550 50  0000 L CNN
 F 1 "0.1uF" H 2400 1450 50  0000 L CNN
-F 2 "" H 2700 1500 50  0001 C CNN
+F 2 "local_footprints:0805_HS" H 2700 1500 50  0001 C CNN
 F 3 "~" H 2700 1500 50  0001 C CNN
 	1    2700 1500
@@
 F 0 "C3" H 3792 1547 50  0000 L CNN
 F 1 "0.1uF" H 3792 1454 50  0000 L CNN
-F 2 "" H 3700 1500 50  0001 C CNN
+F 2 "local_footprints:0805_HS" H 3700 1500 50  0001 C CNN
 F 3 "~" H 3700 1500 50  0001 C CNN
 	1    3700 1500
@@
 F 0 "C4" H 4192 1547 50  0000 L CNN
 F 1 "1uF" H 4192 1454 50  0000 L CNN
-F 2 "" H 4100 1500 50  0001 C CNN
+F 2 "local_footprints:1206_HS" H 4100 1500 50  0001 C CNN
 F 3 "~" H 4100 1500 50  0001 C CNN
 	1    4100 1500
@@
 Connection ~ 4100 1600
 $Comp
-L power:GND #PWR?
+L power:GND #PWR0101
 U 1 1 5C9349E9
 P 4100 1700
-F 0 "#PWR?" H 4100 1450 50  0001 C CNN
+F 0 "#PWR0101" H 4100 1450 50  0001 C CNN
 F 1 "GND" H 4104 1521 50  0000 C CNN
 F 2 "" H 4100 1700 50  0001 C CNN
@@
 F 0 "C5" H 4700 1550 50  0000 L CNN
 F 1 "10uF" H 4600 1450 50  0000 L CNN
-F 2 "" H 4900 1500 50  0001 C CNN
+F 2 "local_footprints:1210_HS" H 4900 1500 50  0001 C CNN
 F 3 "~" H 4900 1500 50  0001 C CNN
 	1    4900 1500
@@
 $EndComp
 $Comp
-L power:GND #PWR?
+L power:GND #PWR0102
 U 1 1 5C934F13
 P 2700 1700
-F 0 "#PWR?" H 2700 1450 50  0001 C CNN
+F 0 "#PWR0102" H 2700 1450 50  0001 C CNN
 F 1 "GND" H 2704 1521 50  0000 C CNN
 F 2 "" H 2700 1700 50  0001 C CNN
@@
 VDD
 $Comp
-L Switch:SW_Push SW_RST
+L Switch:SW_Push SW_RST1
 U 1 1 5C9354AE
 P 1600 2200
-F 0 "SW_RST" V 1650 2650 50  0000 R CNN
+F 0 "SW_RST1" V 1650 2650 50  0000 R CNN
 F 1 "SW_RST" V 1500 2650 50  0000 R CNN
-F 2 "" H 1600 2400 50  0001 C CNN
+F 2 "local_footprints:SW_SPST_PUSH_6mm_3mm" H 1600 2400 50  0001 C CNN
 F 3 "" H 1600 2400 50  0001 C CNN
 	1    1600 2200
@@
 	1600 2400 1600 2500
 $Comp
-L power:GND #PWR?
+L power:GND #PWR0103
 U 1 1 5C935AF9
 P 1600 2500
-F 0 "#PWR?" H 1600 2250 50  0001 C CNN
+F 0 "#PWR0103" H 1600 2250 50  0001 C CNN
 F 1 "GND" H 1604 2321 50  0000 C CNN
 F 2 "" H 1600 2500 50  0001 C CNN
@@
 F 0 "C6" H 1892 2247 50  0000 L CNN
 F 1 "0.1uF" H 1892 2154 50  0000 L CNN
-F 2 "" H 1800 2200 50  0001 C CNN
+F 2 "local_footprints:0805_HS" H 1800 2200 50  0001 C CNN
 F 3 "~" H 1800 2200 50  0001 C CNN
 	1    1800 2200
@@
 Connection ~ 1600 2400
 $Comp
-L Switch:SW_Push SW_BOOT
+L Switch:SW_Push SW_BOOT1
 U 1 1 5C936832
 P 1800 3300
-F 0 "SW_BOOT" V 1850 3750 50  0000 R CNN
+F 0 "SW_BOOT1" V 1850 3750 50  0000 R CNN
 F 1 "SW_BOOT" V 1700 3750 50  0000 R CNN
-F 2 "" H 1800 3500 50  0001 C CNN
+F 2 "local_footprints:SW_SPST_PUSH_6mm_3mm" H 1800 3500 50  0001 C CNN
 F 3 "" H 1800 3500 50  0001 C CNN
 	1    1800 3300
@@
 F 0 "R1" H 1870 3997 50  0000 L CNN
 F 1 "10k" H 1870 3904 50  0000 L CNN
-F 2 "" V 1730 3950 50  0001 C CNN
+F 2 "local_footprints:0805_HS" V 1730 3950 50  0001 C CNN
 F 3 "~" H 1800 3950 50  0001 C CNN
 	1    1800 3950
@@
 	1800 4100 1800 4200
 $Comp
-L power:GND #PWR?
+L power:GND #PWR0104
 U 1 1 5C9382AA
 P 1800 4200
-F 0 "#PWR?" H 1800 3950 50  0001 C CNN
+F 0 "#PWR0104" H 1800 3950 50  0001 C CNN
 F 1 "GND" H 1804 4021 50  0000 C CNN
 F 2 "" H 1800 4200 50  0001 C CNN
@@
 	3300 3800 3300 3900
 $Comp
-L power:GND #PWR?
+L power:GND #PWR0105
 U 1 1 5C93921B
 P 3300 3900
-F 0 "#PWR?" H 3300 3650 50  0001 C CNN
+F 0 "#PWR0105" H 3300 3650 50  0001 C CNN
 F 1 "GND" H 3304 3721 50  0000 C CNN
 F 2 "" H 3300 3900 50  0001 C CNN
@@
 	2700 1600 2700 1700
 $Comp
-L power:GND #PWR?
+L power:GND #PWR0106
 U 1 1 5C940318
 P 4900 1700
-F 0 "#PWR?" H 4900 1450 50  0001 C CNN
+F 0 "#PWR0106" H 4900 1450 50  0001 C CNN
 F 1 "GND" H 4904 1521 50  0000 C CNN
 F 2 "" H 4900 1700 50  0001 C CNN
@@
 F 0 "J1" H 6150 1750 50  0000 L CNN
 F 1 "Conn_01x16" H 5800 1650 50  0000 L CNN
-F 2 "" H 6200 2700 50  0001 C CNN
+F 2 "local_footprints:Pin_Header_Straight_1x16_Pitch2.54mm" H 6200 2700 50  0001 C CNN
 F 3 "~" H 6200 2700 50  0001 C CNN
 	1    6200 2700
@@
 F 0 "J2" H 6650 1750 50  0000 L CNN
 F 1 "Conn_01x16" H 6300 1650 50  0000 L CNN
-F 2 "" H 6700 2700 50  0001 C CNN
+F 2 "local_footprints:Pin_Header_Straight_1x16_Pitch2.54mm" H 6700 2700 50  0001 C CNN
 F 3 "~" H 6700 2700 50  0001 C CNN
 	1    6700 2700
@@
 VDD
 $Comp
-L power:GND #PWR?
+L power:GND #PWR0107
 U 1 1 5C94CD6B
 P 5500 2100
-F 0 "#PWR?" H 5500 1850 50  0001 C CNN
+F 0 "#PWR0107" H 5500 1850 50  0001 C CNN
 F 1 "GND" H 5504 1921 50  0000 C CNN
 F 2 "" H 5500 2100 50  0001 C CNN
@@
 PB7
 $Comp
-L power:GND #PWR?
+L power:GND #PWR0108
 U 1 1 5C95906E
 P 5500 2800
-F 0 "#PWR?" H 5500 2550 50  0001 C CNN
+F 0 "#PWR0108" H 5500 2550 50  0001 C CNN
 F 1 "GND" H 5504 2621 50  0000 C CNN
 F 2 "" H 5500 2800 50  0001 C CNN
@@
 $EndComp
 $Comp
-L power:GND #PWR?
+L power:GND #PWR0109
 U 1 1 5C9598FD
 P 5500 3300
-F 0 "#PWR?" H 5500 3050 50  0001 C CNN
+F 0 "#PWR0109" H 5500 3050 50  0001 C CNN
 F 1 "GND" H 5504 3121 50  0000 C CNN
 F 2 "" H 5500 3300 50  0001 C CNN
@@
 	6900 2600 7500 2600
 $Comp
-L power:GND #PWR?
+L power:GND #PWR0110
 U 1 1 5C95AE32
 P 7500 2600
-F 0 "#PWR?" H 7500 2350 50  0001 C CNN
+F 0 "#PWR0110" H 7500 2350 50  0001 C CNN
 F 1 "GND" H 7504 2421 50  0000 C CNN
 F 2 "" H 7500 2600 50  0001 C CNN
@@
 	6900 3200 7500 3200
 $Comp
-L power:GND #PWR?
+L power:GND #PWR0111
 U 1 1 5C95B168
 P 7500 3200
-F 0 "#PWR?" H 7500 2950 50  0001 C CNN
+F 0 "#PWR0111" H 7500 2950 50  0001 C CNN
 F 1 "GND" H 7504 3021 50  0000 C CNN
 F 2 "" H 7500 3200 50  0001 C CNN
@@
 	6900 2000 7500 2000
 $Comp
-L power:GND #PWR?
+L power:GND #PWR0112
 U 1 1 5C95BB28
 P 7500 2000
-F 0 "#PWR?" H 7500 1750 50  0001 C CNN
+F 0 "#PWR0112" H 7500 1750 50  0001 C CNN
 F 1 "GND" H 7504 1821 50  0000 C CNN
 F 2 "" H 7500 2000 50  0001 C CNN

Commit message: Added optional battery connector and 2V5 regulator
Parts:
- added C7, C8: 0.1u, local_footprints:0805_HS, symbol Device:C_Small
- added J3: JST_PH, local_footprints:JST_PH_S2B-PH-K_02x2.00mm_Angled_WiderHole, symbol Connector_Generic:Conn_01x02
- added U2: AP7354, local_footprints:SOT-23-5_HS, symbol local_symbols:AP7354
Connections:
- net GND: now also C7.1, C8.2, J3.2 (Pin_2), U2.2 (GND)
- net VDD: now also C8.1, U2.5 (VOUT)
- new net: C7.2, J3.1 (Pin_1), U2.1 (VIN), U2.3 (EN)
Other:
- note added: "Optional battery input (JST PH 2.0mm)\nwith low-power 2.5V regulator."
- moved on the sheet: C1, C2, C3, C4, C5, C6, J1, J2, R1, SW_BOOT1, SW_RST1, U1
