File: stm32l031-breakout.kicad_pcb (KiCad board)
At the start: 2 copper layers, 0 parts

Commit message: Footprint tuning, net list, initial PCB placement
Parts:
- added C1: 0.1uF, local_footprints:0805_HS, F.Cu at (151.1, 111.8)
- added C2: 0.1uF, local_footprints:0805_HS, F.Cu at (166.4, 111.8)
- added C3: 0.1uF, local_footprints:0805_HS, F.Cu at (153.2, 116.4)
- added C4: 1uF, local_footprints:1206_HS, F.Cu at (149.9, 116.8)
- added C5: 10uF, local_footprints:1210_HS, F.Cu at (141.0, 119.4)
- added C6: 0.1uF, local_footprints:0805_HS, F.Cu at (139.7, 105.4)
- added J1: Conn_01x16, local_footprints:Pin_Header_Straight_1x16_Pitch2.54mm, F.Cu at (139.7, 121.9)
- added J2: Conn_01x16, local_footprints:Pin_Header_Straight_1x16_Pitch2.54mm, F.Cu at (139.7, 101.6)
- added R1: 10k, local_footprints:0805_HS, F.Cu at (144.8, 105.4)
- added SW_BOOT1: SW_BOOT, local_footprints:SW_SPST_PUSH_6mm_3mm, F.Cu at (144.8, 111.8)
- added SW_RST1: SW_RST, local_footprints:SW_SPST_PUSH_6mm_3mm, F.Cu at (139.7, 111.8)
- added U1: STM32L031K6Tx, local_footprints:TQFP-32_7x7mm_Pitch0.8mm_HS_narrow_pads, F.Cu at (158.8, 111.8)
